File: pcb/piracer_evo_mainboard/piracer_evo_mainboard.kicad_pcb (KiCad board)
At the start: 2 copper layers, 125 x 104.5 mm, 23 parts, among them J1 PiRacer-BoardConnector, J2 PiRacer-BoardConnector, J3 Conn_01x03, J4 Conn_01x03, U1 PCA9685PW

Commit message: First complete version
Parts:
- removed the REF** at (257.5, 157.0)
- removed the REF** at (200.2, 126.2)
- added ?: , , F.Cu at (178.2, 116.5)
- added ?: , , F.Cu at (257.5, 165.2)
- added ?: , , F.Cu at (204.2, 119.0)
- added ?: , , F.Cu at (199.0, 126.5)
- added ?: , , F.Cu at (250.0, 78.0)
- added C2: 22pF, Capacitor_SMD:C_0805_2012Metric_Pad1.18x1.45mm_HandSolder, B.Cu at (173.2, 120.5)
- added C3: 22pF, Capacitor_SMD:C_0805_2012Metric_Pad1.18x1.45mm_HandSolder, B.Cu at (178.2, 120.5)
- added C4: 22pF, Capacitor_SMD:C_0805_2012Metric_Pad1.18x1.45mm_HandSolder, B.Cu at (238.0, 119.8)
- added C5: 22pF, Capacitor_SMD:C_0805_2012Metric_Pad1.18x1.45mm_HandSolder, B.Cu at (243.0, 119.8)
- added C6: 100nF, Capacitor_SMD:C_0805_2012Metric_Pad1.18x1.45mm_HandSolder, B.Cu at (165.0, 129.0)
- added C7: 100nF, Capacitor_SMD:C_0805_2012Metric_Pad1.18x1.45mm_HandSolder, B.Cu at (229.5, 130.0)
- added J10: Extension_Front, Connector_JST:JST_EH_S5B-EH_1x05_P2.50mm_Horizontal, B.Cu at (176.0, 79.5)
- added J11: Extension_Rear, Connector_JST:JST_EH_S5B-EH_1x05_P2.50mm_Horizontal, B.Cu at (147.5, 170.5)
- added J12: Debug_BreadBoard, Connector_PinHeader_2.54mm:PinHeader_2x03_P2.54mm_Vertical, F.Cu at (195.7, 168.7)
- added J13: Debug_Power, Connector_PinHeader_2.54mm:PinHeader_1x03_P2.54mm_Horizontal, B.Cu at (148.1, 103.7)
- added J14: Debug_CAN, Connector_PinHeader_2.54mm:PinHeader_1x03_P2.54mm_Horizontal, B.Cu at (251.9, 114.0)
- added J15: Debug_Bat, Connector_PinHeader_2.54mm:PinHeader_1x05_P2.54mm_Horizontal, B.Cu at (148.1, 87.9)
- added J16: Debug_RC, Connector_PinHeader_2.54mm:PinHeader_1x04_P2.54mm_Horizontal, B.Cu at (252.1, 156.6)
- added J17: Debug_I2C, Connector_PinHeader_2.54mm:PinHeader_1x03_P2.54mm_Horizontal, B.Cu at (252.1, 96.0)
- added J18: Input_BatBalancer, Connector_JST:JST_EH_B4B-EH-A_1x04_P2.50mm_Vertical, B.Cu at (154.8, 87.0)
- added J19: CAN_Term_Jumper, Connector_PinHeader_2.54mm:PinHeader_1x02_P2.54mm_Vertical, F.Cu at (167.2, 89.8)
- added J7: Input_RC1, Connector_PinHeader_2.54mm:PinHeader_1x03_P2.54mm_Vertical, B.Cu at (209.3, 123.8)
- added J8: Input_RC2, Connector_PinHeader_2.54mm:PinHeader_1x03_P2.54mm_Vertical, B.Cu at (209.3, 127.5)
- added J9: Input_RC3, Connector_PinHeader_2.54mm:PinHeader_1x03_P2.54mm_Vertical, B.Cu at (209.3, 131.2)
- added R3: 10K, Resistor_SMD:R_1206_3216Metric_Pad1.30x1.75mm_HandSolder, B.Cu at (168.2, 142.8)
- added R4: 10K, Resistor_SMD:R_1206_3216Metric_Pad1.30x1.75mm_HandSolder, B.Cu at (233.2, 142.8)
- added R5: 0-100k, Resistor_SMD:R_1206_3216Metric_Pad1.30x1.75mm_HandSolder, B.Cu at (167.8, 116.8)
- added R6: 0-100k, Resistor_SMD:R_1206_3216Metric_Pad1.30x1.75mm_HandSolder, B.Cu at (232.2, 117.8)
- added R7: 60, Resistor_SMD:R_1206_3216Metric_Pad1.30x1.75mm_HandSolder, B.Cu at (170.0, 85.2)
- added REF**: via_0.9, twyleg-misc:via_0.9, F.Cu at (154.2, 93.0)
- added U2: MCP2515-xSO, Package_SO:SOIC-18W_7.5x11.6mm_P1.27mm, B.Cu at (172.8, 135.2)
- added U3: MCP2515-xSO, Package_SO:SOIC-18W_7.5x11.6mm_P1.27mm, B.Cu at (237.2, 135.2)
- added U4: SN65HVD231, Package_SO:SOIC-8_3.9x4.9mm_P1.27mm, B.Cu at (165.8, 123.2)
- added U5: SN65HVD231, Package_SO:SOIC-8_3.9x4.9mm_P1.27mm, B.Cu at (230.2, 124.2)
- added Y1: 16MHz, Crystal:Crystal_HC18-U_Vertical, F.Cu at (173.3, 125.8)
- added Y2: 16MHz, Crystal:Crystal_HC18-U_Vertical, F.Cu at (238.1, 124.8)
- J1: footprint twyleg-board-connectors:RaspberryPi3-ModelB-Power+I2C -> twyleg-board-connectors:RaspberryPi3-ModelB-PiracerEvo
- J2: footprint twyleg-board-connectors:Arduino_UNO_R3_WithMountingHoles-Power+I2C -> twyleg-board-connectors:Arduino_UNO_R3_WithMountingHoles-PiRacerEvo
- J3: value Conn_01x03 -> Output_Servo
- J4: value Conn_01x03 -> Output_ESC
- J5: renamed from BAT-In1; value T-Plug -> Power_Bat
- J6: renamed from DriveTrain-Out1; value T-Plug -> Power_DriveTrain
- moved U1 5.50 mm to (219.0, 138.5)
- moved R2 4.00 mm to (222.5, 129.5), turned to 180 degrees
- moved R1 3.75 mm to (217.5, 129.5)
- moved REF** 0.50 mm to (211.5, 87.2)
- moved ? 0.35 mm to (258.5, 126.0)
Connections:
- R2 pad 1: /SCL -> /+3V3
- R2 pad 2: /+3V3 -> /SCL
- REF** pad : (no net) -> /GND
Routing:
- net /+3V3: track 273.7 -> 528.5 mm
- net /CAN_H: track 0.00 -> 253.7 mm, vias 0 -> 2
- net /CAN_L: track 0.00 -> 253.3 mm, vias 0 -> 2
- net /+5V: track 184.1 -> 363.0 mm, vias 0 -> 3
- net /VBAT_C3: track 0.00 -> 172.2 mm, vias 0 -> 1
- net /VBAT+: track 56.1 -> 226.5 mm, vias 1 -> 3
- net /VBAT_C2: track 0.00 -> 169.3 mm, vias 0 -> 1
- net /VBAT_C1: track 0.00 -> 162.6 mm, vias 0 -> 1
- net /RC_1: track 0.00 -> 81.8 mm
- net /RC_2: track 0.00 -> 68.6 mm
- net /SDA: track 192.1 -> 255.9 mm
- net /RC_3: track 0.00 -> 58.7 mm
- net /SCL: track 183.9 -> 229.0 mm
- net /MISO_A: track 0.00 -> 28.6 mm
- net /CAN_CS_A: track 0.00 -> 27.9 mm
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