File: pcb/piracer_evo_mainboard/piracer_evo_mainboard.kicad_sch (KiCad schematic)
At the start: 3 parts

Commit message: 90% complete version
Parts:
- removed J? (x2): Conn_01x02, symbol Connector_Generic:Conn_01x02
- removed J?: Raspberry_Pi_2_3, symbol Connector:Raspberry_Pi_2_3
- added A1: Adafruit_IMU_BNO055, twyleg-board-connectors:Adafruit_IMU_BNO055, symbol twyleg-board-connectors:Adafruit_IMU_BNO055
- added A2: Waveshare-0_96inch-oled, twyleg-displays:Waveshare-0_96inch-oled, symbol twyleg-board-connectors:Waveshare-0_96inch-oled
- added BAT-In1: T-Plug, twyleg-connectors:T-Plug-Male, symbol twyleg-connectors:T-Plug
- added C1: C, symbol Device:C
- added DriveTrain-Out1: T-Plug, twyleg-connectors:T-Plug-Female, symbol twyleg-connectors:T-Plug
- added J1: PiRacer-BoardConnector, twyleg-board-connectors:RaspberryPi3-ModelB-Power+I2C, symbol twyleg-board-connectors:PiRacer-BoardConnector
- added J2: PiRacer-BoardConnector, twyleg-board-connectors:Arduino_UNO_R3_WithMountingHoles-Power+I2C, symbol twyleg-board-connectors:PiRacer-BoardConnector
- added J3, J4: Conn_01x03, Connector_PinHeader_2.54mm:PinHeader_1x03_P2.54mm_Vertical, symbol Connector_Generic:Conn_01x03
- added PS1: Polulu-S13V30F5, twyleg-voltage-regulators:Polulu-S13V30F5, symbol twyleg-voltage-regulators:Polulu-S13V30F5
- added R1, R2: 4.7K, Resistor_SMD:R_1206_3216Metric_Pad1.30x1.75mm_HandSolder, symbol Device:R
- added U1: PCA9685PW, Package_SO:TSSOP-28_4.4x9.7mm_P0.65mm, symbol Driver_LED:PCA9685PW
Connections:
- new net +3V3: A1.5 (VIN), A2.1 (RES), A2.8 (VCC), C1.1, J1.1 (+3V3), J2.1 (+3V3), R1.1, R2.2, U1.28 (VDD)
- new net +5V: J1.2 (+5V), J1.4 (+5V), J2.2 (+5V), J2.4 (+5V), PS1.1 (VOUT)
- new net ESC_+5V: J3.2 (Pin_2), J4.2 (Pin_2)
- new net ESC_PWM: J4.1 (Pin_1), U1.7 (LED1)
- new net GND: A1.7 (GND), A2.3 (CS), A2.7 (GND), BAT-In1.2 (-), C1.2, DriveTrain-Out1.2 (-), J1.6 (GND), J2.6 (GND), J3.3 (Pin_3), J4.3 (Pin_3), PS1.2 (GND), PS1.3 (GND), U1.1 (A0), U1.14 (VSS), U1.2 (A1), U1.23 (~{OE}), U1.24 (A5), U1.25 (EXTCLK), U1.3 (A2), U1.4 (A3), U1.5 (A4)
- new net SCL: A1.9 (SCL), A2.4 (CLK), J1.5 (SCL), J2.5 (SCL), R2.1, U1.26 (SCL)
- new net SDA: A1.8 (SDA), A2.5 (DIN), J1.3 (SDA), J2.3 (SDA), R1.2, U1.27 (SDA)
- new net SERVO_PWM: J3.1 (Pin_1), U1.6 (LED0)
- new net VBAT+: BAT-In1.1 (+), DriveTrain-Out1.1 (+), PS1.4 (VIN)
- no-connect marks 0 -> 22

Commit message: First complete version
Parts:
- removed C1: C, symbol Device:C
- added C2, C3, C4, C5: 22pF, Capacitor_SMD:C_0805_2012Metric_Pad1.18x1.45mm_HandSolder, symbol Device:C
- added C6, C7: 100nF, Capacitor_SMD:C_0805_2012Metric_Pad1.18x1.45mm_HandSolder, symbol Device:C
- added J10: Extension_Front, Connector_JST:JST_EH_S5B-EH_1x05_P2.50mm_Horizontal, symbol Connector_Generic:Conn_01x05
- added J11: Extension_Rear, Connector_JST:JST_EH_S5B-EH_1x05_P2.50mm_Horizontal, symbol Connector_Generic:Conn_01x05
- added J12: Debug_BreadBoard, Connector_PinHeader_2.54mm:PinHeader_2x03_P2.54mm_Vertical, symbol Connector_Generic:Conn_02x03_Odd_Even
- added J13: Debug_Power, Connector_PinHeader_2.54mm:PinHeader_1x03_P2.54mm_Horizontal, symbol Connector_Generic:Conn_01x03
- added J14: Debug_CAN, Connector_PinHeader_2.54mm:PinHeader_1x03_P2.54mm_Horizontal, symbol Connector_Generic:Conn_01x03
- added J15: Debug_Bat, Connector_PinHeader_2.54mm:PinHeader_1x05_P2.54mm_Horizontal, symbol Connector_Generic:Conn_01x05
- added J16: Debug_RC, Connector_PinHeader_2.54mm:PinHeader_1x04_P2.54mm_Horizontal, symbol Connector_Generic:Conn_01x04
- added J17: Debug_I2C, Connector_PinHeader_2.54mm:PinHeader_1x03_P2.54mm_Horizontal, symbol Connector_Generic:Conn_01x03
- added J18: Input_BatBalancer, Connector_JST:JST_EH_B4B-EH-A_1x04_P2.50mm_Vertical, symbol Connector_Generic:Conn_01x04
- added J19: CAN_Term_Jumper, Connector_PinHeader_2.54mm:PinHeader_1x02_P2.54mm_Vertical, symbol Connector_Generic:Conn_01x02
- added J7: Input_RC1, Connector_PinHeader_2.54mm:PinHeader_1x03_P2.54mm_Vertical, symbol Connector_Generic:Conn_01x03
- added J8: Input_RC2, Connector_PinHeader_2.54mm:PinHeader_1x03_P2.54mm_Vertical, symbol Connector_Generic:Conn_01x03
- added J9: Input_RC3, Connector_PinHeader_2.54mm:PinHeader_1x03_P2.54mm_Vertical, symbol Connector_Generic:Conn_01x03
- added R3, R4: 10K, Resistor_SMD:R_1206_3216Metric_Pad1.30x1.75mm_HandSolder, symbol Device:R
- added R5, R6: 0-100k, Resistor_SMD:R_1206_3216Metric_Pad1.30x1.75mm_HandSolder, symbol Device:R
- added R7: 60, Resistor_SMD:R_1206_3216Metric_Pad1.30x1.75mm_HandSolder, symbol Device:R
- added U2, U3: MCP2515-xSO, Package_SO:SOIC-18W_7.5x11.6mm_P1.27mm, symbol Interface_CAN_LIN:MCP2515-xSO
- added U4, U5: SN65HVD231, Package_SO:SOIC-8_3.9x4.9mm_P1.27mm, symbol Interface_CAN_LIN:SN65HVD231
- added Y1, Y2: 16MHz, Crystal:Crystal_HC18-U_Vertical, symbol Device:Crystal
- J3: value Conn_01x03 -> Output_Servo
- J4: value Conn_01x03 -> Output_ESC
- J5: renamed from BAT-In1; value T-Plug -> Power_Bat
- J6: renamed from DriveTrain-Out1; value T-Plug -> Power_DriveTrain
Connections:
- net +3V3: now also R2.1, C6.2, C7.2, J10.3 (Pin_3), J11.3 (Pin_3), J12.3 (Pin_3), J13.3 (Pin_3), R3.2, R4.2, U2.18 (VDD), U3.18 (VDD), U4.3 (VCC), U5.3 (VCC); no longer R2.2
- net +5V: now also J10.2 (Pin_2), J11.2 (Pin_2), J12.1 (Pin_1), J13.1 (Pin_1), J7.2 (Pin_2), J8.2 (Pin_2), J9.2 (Pin_2)
- net GND: now also C2.1, C3.1, C4.1, C5.1, C6.1, C7.1, J10.1 (Pin_1), J11.1 (Pin_1), J12.2 (Pin_2), J12.4 (Pin_4), J13.2 (Pin_2), J14.2 (Pin_2), J15.1 (Pin_1), J16.1 (Pin_1), J17.1 (Pin_1), J18.4 (Pin_4), J7.3 (Pin_3), J8.3 (Pin_3), J9.3 (Pin_3), R5.1, R6.1, U2.9 (VSS), U3.9 (VSS), U4.2 (GND), U5.2 (GND)
- net SCL: now also R2.2, J12.6 (Pin_6), J17.2 (Pin_2); no longer R2.1
- net SDA: now also J12.5 (Pin_5), J17.3 (Pin_3)
- net VBAT+: now also J2.8 (BAT), J15.2 (Pin_2)
- new net: C2.2, U2.7 (OSC2), Y1.1
- new net: C3.2, U2.8 (OSC1), Y1.2
- new net: R4.1, U3.17 (~{RESET})
- new net: C4.2, U3.7 (OSC2), Y2.1
- new net: C5.2, U3.8 (OSC1), Y2.2
- new net: R5.2, U4.8 (Rs)
- new net: J19.2 (Pin_2), R7.1
- new net: R3.1, U2.17 (~{RESET})
- new net: R6.2, U5.8 (Rs)
- new net CAN_CS_A: J1.13 (CAN_CS), U2.16 (~{CS})
- new net CAN_CS_B: J2.13 (CAN_CS), U3.16 (~{CS})
- new net CAN_H: J10.4 (Pin_4), J11.4 (Pin_4), J14.1 (Pin_1), R7.2, U4.7 (CANH), U5.7 (CANH)
- new net CAN_INT_A: J1.15 (CAN_INT), U2.12 (~{INT})
- new net CAN_INT_B: J2.15 (CAN_INT), U3.12 (~{INT})
- new net CAN_L: J10.5 (Pin_5), J11.5 (Pin_5), J14.3 (Pin_3), J19.1 (Pin_1), U4.6 (CANL), U5.6 (CANL)
- new net CAN_RX_A: U2.2 (RXCAN), U4.4 (R)
- new net CAN_RX_B: U3.2 (RXCAN), U5.4 (R)
- new net CAN_TX_A: U2.1 (TXCAN), U4.1 (D)
- new net CAN_TX_B: U3.1 (TXCAN), U5.1 (D)
- new net MISO_A: J1.7 (MISO), U2.15 (SO)
- new net MISO_B: J2.7 (MISO), U3.15 (SO)
- new net MOSI_A: J1.9 (MOSI), U2.14 (SI)
- new net MOSI_B: J2.9 (MOSI), U3.14 (SI)
- new net RC_1: J16.2 (Pin_2), J2.16 (RC_CH1), J7.1 (Pin_1)
- new net RC_2: J16.3 (Pin_3), J2.17 (RC_CH2), J8.1 (Pin_1)
- new net RC_3: J16.4 (Pin_4), J2.18 (RC_CH3), J9.1 (Pin_1)
- new net SCK_A: J1.11 (CLK), U2.13 (SCK)
- new net SCK_B: J2.11 (CLK), U3.13 (SCK)
- new net VBAT_C1: J15.3 (Pin_3), J18.3 (Pin_3), J2.10 (BAT_C1)
- new net VBAT_C2: J15.4 (Pin_4), J18.2 (Pin_2), J2.12 (BAT_C2)
- new net VBAT_C3: J15.5 (Pin_5), J18.1 (Pin_1), J2.14 (BAT_C3)
- no-connect marks 22 -> 43
Other:
- moved on the sheet: A1, A2, J3, J4, J5, J6, PS1, R1, R2, U1
